File: pcb/tiny-sao.sch (KiCad schematic (older format))
At the start: 5 parts, among them J1 Conn_02x02_Counter_Clockwise, SW1 SW_Push, U1 ATtiny45-20SU

Commit message: fix(pcb): SCL and SDA were crossed
Parts:
- J1: value Conn_02x02_Counter_Clockwise -> Male_02x02; symbol Connector_Generic:Conn_02x02_Counter_Clockwise -> Connector_Generic:Conn_02x02_Top_Bottom
Changed lines of the file:
@@
 EESchema Schematic File Version 4
 LIBS:tiny-sao-cache
-EELAYER 26 0
+EELAYER 29 0
 EELAYER END
 $Descr A4 11693 8268
@@
 $EndComp
 $Comp
-L Connector_Generic:Conn_02x02_Counter_Clockwise J1
+L Connector_Generic:Conn_02x02_Top_Bottom J1
 U 1 1 5C488EC3
 P 7150 3600
 F 0 "J1" H 7200 3817 50  0000 C CNN
-F 1 "Conn_02x02_Counter_Clockwise" H 7200 3726 50  0000 C CNN
+F 1 "Male_02x02" H 7200 3726 50  0000 C CNN
 F 2 "Connector_PinHeader_2.54mm:PinHeader_2x02_P2.54mm_Vertical" H 7150 3600 50  0001 C CNN
 F 3 "~" H 7150 3600 50  0001 C CNN
